Commit message: edited the number of joints to be 7 and edited the auto navigation to be using a slider instead of hardcoded

File: src/smart_endoscope/urdf/smart_broncho.urdf (robot description, URDF)
Before this commit: robot bronchoscope, 6 links, 5 joints
Links:
- removed link mid_link1
- removed link mid_link2
- added link link_1, mass 0.2; collision cylinder length=0.1 radius=0.014; visual cylinder length=0.1 radius=0.014
- added link link_2, mass 0.2; collision cylinder length=0.1 radius=0.013; visual cylinder length=0.1 radius=0.013
- added link link_3, mass 0.2; collision cylinder length=0.1 radius=0.013; visual cylinder length=0.1 radius=0.013
- added link link_4, mass 0.2; collision cylinder length=0.1 radius=0.012; visual cylinder length=0.1 radius=0.012
- added link link_5, mass 0.1; collision cylinder length=0.05 radius=0.012; visual cylinder length=0.05 radius=0.012
- link distal_tip: mass 1.0 -> 0.1; geometry collision cylinder length=0.05 radius=0.012; collision sphere radius=0.012
Joints:
- removed joint distal_joint
- removed joint mid_joint
- removed joint proximal_joint
- added joint distal_roll_joint: type revolute, parent link_5, child distal_tip, origin xyz=0.05 0 0 rpy=0 0 0, axis 1 0 0, limit lower=-3.14 upper=3.14 effort=50.0 velocity=2.0
- added joint distal_yaw_joint: type revolute, parent link_4, child link_5, origin xyz=0.1 0 0 rpy=0 0 0, axis 0 0 1, limit lower=-1.57 upper=1.57 effort=100.0 velocity=1.0
- added joint mid_pitch_joint: type revolute, parent link_3, child link_4, origin xyz=0.1 0 0 rpy=0 0 0, axis 0 1 0, limit lower=-1.0 upper=1.0 effort=100.0 velocity=1.0
- added joint mid_yaw_joint: type revolute, parent link_2, child link_3, origin xyz=0.1 0 0 rpy=0 0 0, axis 0 0 1, limit lower=-1.0 upper=1.0 effort=100.0 velocity=1.0
- added joint proximal_pitch_joint: type revolute, parent link_1, child link_2, origin xyz=0.1 0 0 rpy=0 0 0, axis 0 1 0, limit lower=-0.6 upper=0.6 effort=100.0 velocity=1.0
- added joint proximal_yaw_joint: type revolute, parent base_link, child link_1, origin xyz=0 0 0 rpy=0 0 0, axis 0 0 1, limit lower=-0.6 upper=0.6 effort=100.0 velocity=1.0

Commit message: enabled up and down movements for the whole robot

File: src/smart_endoscope/urdf/smart_broncho.urdf (robot description, URDF)
Before this commit: robot bronchoscope, 9 links, 8 joints
Links:
- added link vertical_carriage, mass 0.5
- link rail_link: mass 1.0 -> 2.0
Joints:
- added joint vertical_joint: type prismatic, parent rail_link, child vertical_carriage, origin xyz=0 0 0 rpy=0 0 0, axis 0 0 1, limit lower=-0.3 upper=0.3 effort=100.0 velocity=0.5
- joint insertion_joint: parent rail_link -> vertical_carriage
